File: pad/pad.kicad_pcb (KiCad board)
At the start: 2 copper layers, 110 x 133 mm, 44 parts, among them J1 OLED_128x64, SW1 ESC, SW10 5, SW11 6, SW12 1, SW13 2, SW14 3, SW15 entrt, SW16 0, SW17 ., SW18 RotaryEncoder_Switch, SW19 RotaryEncoder_Switch, SW2 /, SW3 *, SW4 -, SW5 7, SW6 8, SW7 9, SW8 +, SW9 4, U1 Raspberry_Pi_Pico

Commit message: BOM
Parts:
- added H4: MountingHole, MountingHole:MountingHole_3.2mm_M3, F.Cu at (3.48, 3.48)
Connections:
- U1 pad 13: Row5 -> unconnected-(U1-GND-Pad13)
- U1 pad 14: unconnected-(U1-GPIO10-Pad14) -> Row5
Routing:
- net Row5: track 150.5 -> 148.0 mm
Changed lines of the file:
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@@
 	(net 49 "unconnected-(U1-SWDIO-Pad43)")
 	(net 50 "unconnected-(U1-GPIO26_ADC0-Pad31)")
-	(net 51 "unconnected-(U1-GPIO10-Pad14)")
-	(net 52 "unconnected-(U1-3V3_EN-Pad37)")
-	(net 53 "unconnected-(U1-ADC_VREF-Pad35)")
-	(net 54 "unconnected-(U1-GPIO2-Pad4)")
-	(net 55 "unconnected-(U1-GND-Pad18)")
-	(net 56 "unconnected-(U1-GPIO27_ADC1-Pad32)")
-	(net 57 "unconnected-(U1-GPIO1-Pad2)")
-	(net 58 "unconnected-(U1-GND-Pad38)")
-	(net 59 "unconnected-(U1-GPIO28_ADC2-Pad34)")
-	(net 60 "unconnected-(U1-RUN-Pad30)")
-	(net 61 "unconnected-(U1-GPIO9-Pad12)")
-	(net 62 "unconnected-(U1-AGND-Pad33)")
-	(net 63 "unconnected-(U1-GPIO15-Pad20)")
-	(net 64 "unconnected-(U1-GND-Pad42)")
+	(net 51 "unconnected-(U1-3V3_EN-Pad37)")
+	(net 52 "unconnected-(U1-ADC_VREF-Pad35)")
+	(net 53 "unconnected-(U1-GPIO2-Pad4)")
+	(net 54 "unconnected-(U1-GND-Pad18)")
+	(net 55 "unconnected-(U1-GPIO27_ADC1-Pad32)")
+	(net 56 "unconnected-(U1-GPIO1-Pad2)")
+	(net 57 "unconnected-(U1-GND-Pad38)")
+	(net 58 "unconnected-(U1-GPIO28_ADC2-Pad34)")
+	(net 59 "unconnected-(U1-RUN-Pad30)")
+	(net 60 "unconnected-(U1-GPIO9-Pad12)")
+	(net 61 "unconnected-(U1-AGND-Pad33)")
+	(net 62 "unconnected-(U1-GPIO15-Pad20)")
+	(net 63 "unconnected-(U1-GND-Pad42)")
+	(net 64 "unconnected-(U1-GND-Pad13)")
 	(footprint "ScottoKeebs_MX:MX_PCB_1.00u"
 		(layer "F.Cu")
@@
 			(layers "*.Cu" "*.Mask")
 			(remove_unused_layers no)
-			(net 57 "unconnected-(U1-GPIO1-Pad2)")
+			(net 56 "unconnected-(U1-GPIO1-Pad2)")
 			(pinfunction "GPIO1")
 			(pintype "bidirectional")
@@
 			)
 			(layers "F.Cu" "F.Mask")
-			(net 57 "unconnected-(U1-GPIO1-Pad2)")
+			(net 56 "unconnected-(U1-GPIO1-Pad2)")
 			(pinfunction "GPIO1")
 			(pintype "bidirectional")
@@
 			(layers "*.Cu" "*.Mask")
 			(remove_unused_layers no)
-			(net 54 "unconnected-(U1-GPIO2-Pad4)")
+			(net 53 "unconnected-(U1-GPIO2-Pad4)")
 			(pinfunction "GPIO2")
 			(pintype "bidirectional")
@@
 			)
 			(layers "F.Cu" "F.Mask")
-			(net 54 "unconnected-(U1-GPIO2-Pad4)")
+			(net 53 "unconnected-(U1-GPIO2-Pad4)")
 			(pinfunction "GPIO2")
 			(pintype "bidirectional")
@@
 			(layers "*.Cu" "*.Mask")
 			(remove_unused_layers no)
-			(net 61 "unconnected-(U1-GPIO9-Pad12)")
+			(net 60 "unconnected-(U1-GPIO9-Pad12)")
 			(pinfunction "GPIO9")
 			(pintype "bidirectional")
@@
 			)
 			(layers "F.Cu" "F.Mask")
-			(net 61 "unconnected-(U1-GPIO9-Pad12)")
+			(net 60 "unconnected-(U1-GPIO9-Pad12)")
 			(pinfunction "GPIO9")
 			(pintype "bidirectional")
@@
 			(layers "*.Cu" "*.Mask")
 			(remove_unused_layers no)
-			(net 15 "Row5")
+			(net 64 "unconnected-(U1-GND-Pad13)")
 			(pinfunction "GND")
 			(pintype "power_in")
@@
 			)
 			(layers "F.Cu" "F.Mask")
-			(net 15 "Row5")
+			(net 64 "unconnected-(U1-GND-Pad13)")
 			(pinfunction "GND")
 			(pintype "power_in")
@@
 			(layers "*.Cu" "*.Mask")
 			(remove_unused_layers no)
-			(net 51 "unconnected-(U1-GPIO10-Pad14)")
+			(net 15 "Row5")
 			(pinfunction "GPIO10")
 			(pintype "bidirectional")
@@
 			)
 			(layers "F.Cu" "F.Mask")
-			(net 51 "unconnected-(U1-GPIO10-Pad14)")
+			(net 15 "Row5")
 			(pinfunction "GPIO10")
 			(pintype "bidirectional")
@@
 			(layers "*.Cu" "*.Mask")
 			(remove_unused_layers no)
-			(net 55 "unconnected-(U1-GND-Pad18)")
+			(net 54 "unconnected-(U1-GND-Pad18)")
 			(pinfunction "GND")
 			(pintype "power_in")
@@
 			)
 			(layers "F.Cu" "F.Mask")
-			(net 55 "unconnected-(U1-GND-Pad18)")
+			(net 54 "unconnected-(U1-GND-Pad18)")
 			(pinfunction "GND")
 			(pintype "power_in")
@@
 			(layers "*.Cu" "*.Mask")
 			(remove_unused_layers no)
-			(net 63 "unconnected-(U1-GPIO15-Pad20)")
+			(net 62 "unconnected-(U1-GPIO15-Pad20)")
 			(pinfunction "GPIO15")
 			(pintype "bidirectional")
@@
 			)
 			(layers "F.Cu" "F.Mask")
-			(net 63 "unconnected-(U1-GPIO15-Pad20)")
+			(net 62 "unconnected-(U1-GPIO15-Pad20)")
 			(pinfunction "GPIO15")
 			(pintype "bidirectional")
@@
 			(layers "*.Cu" "*.Mask")
 			(remove_unused_layers no)
-			(net 60 "unconnected-(U1-RUN-Pad30)")
+			(net 59 "unconnected-(U1-RUN-Pad30)")
 			(pinfunction "RUN")
 			(pintype "input")
@@
 			)
 			(layers "F.Cu" "F.Mask")
-			(net 60 "unconnected-(U1-RUN-Pad30)")
+			(net 59 "unconnected-(U1-RUN-Pad30)")
 			(pinfunction "RUN")
 			(pintype "input")
@@
 			(layers "*.Cu" "*.Mask")
 			(remove_unused_layers no)
-			(net 56 "unconnected-(U1-GPIO27_ADC1-Pad32)")
+			(net 55 "unconnected-(U1-GPIO27_ADC1-Pad32)")
 			(pinfunction "GPIO27_ADC1")
 			(pintype "bidirectional")
@@
 			)
 			(layers "F.Cu" "F.Mask")
-			(net 56 "unconnected-(U1-GPIO27_ADC1-Pad32)")
+			(net 55 "unconnected-(U1-GPIO27_ADC1-Pad32)")
 			(pinfunction "GPIO27_ADC1")
 			(pintype "bidirectional")
@@
 			(layers "*.Cu" "*.Mask")
 			(remove_unused_layers no)
-			(net 62 "unconnected-(U1-AGND-Pad33)")
+			(net 61 "unconnected-(U1-AGND-Pad33)")
 			(pinfunction "AGND")
 			(pintype "power_in")
@@
 			)
 			(layers "F.Cu" "F.Mask")
-			(net 62 "unconnected-(U1-AGND-Pad33)")
+			(net 61 "unconnected-(U1-AGND-Pad33)")
 			(pinfunction "AGND")
 			(pintype "power_in")
@@
 			(layers "*.Cu" "*.Mask")
 			(remove_unused_layers no)
-			(net 59 "unconnected-(U1-GPIO28_ADC2-Pad34)")
+			(net 58 "unconnected-(U1-GPIO28_ADC2-Pad34)")
 			(pinfunction "GPIO28_ADC2")
 			(pintype "bidirectional")
@@
 			)
 			(layers "F.Cu" "F.Mask")
-			(net 59 "unconnected-(U1-GPIO28_ADC2-Pad34)")
+			(net 58 "unconnected-(U1-GPIO28_ADC2-Pad34)")
 			(pinfunction "GPIO28_ADC2")
 			(pintype "bidirectional")
@@
 			(layers "*.Cu" "*.Mask")
 			(remove_unused_layers no)
-			(net 53 "unconnected-(U1-ADC_VREF-Pad35)")
+			(net 52 "unconnected-(U1-ADC_VREF-Pad35)")
 			(pinfunction "ADC_VREF")
 			(pintype "power_in")
@@
 			)
 			(layers "F.Cu" "F.Mask")
-			(net 53 "unconnected-(U1-ADC_VREF-Pad35)")
+			(net 52 "unconnected-(U1-ADC_VREF-Pad35)")
 			(pinfunction "ADC_VREF")
 			(pintype "power_in")
@@
 			(layers "*.Cu" "*.Mask")
 			(remove_unused_layers no)
-			(net 52 "unconnected-(U1-3V3_EN-Pad37)")
+			(net 51 "unconnected-(U1-3V3_EN-Pad37)")
 			(pinfunction "3V3_EN")
 			(pintype "input")
@@
 			)
 			(layers "F.Cu" "F.Mask")
-			(net 52 "unconnected-(U1-3V3_EN-Pad37)")
+			(net 51 "unconnected-(U1-3V3_EN-Pad37)")
 			(pinfunction "3V3_EN")
 			(pintype "input")
@@
 			(layers "*.Cu" "*.Mask")
 			(remove_unused_layers no)
-			(net 58 "unconnected-(U1-GND-Pad38)")
+			(net 57 "unconnected-(U1-GND-Pad38)")
 			(pinfunction "GND")
 			(pintype "bidirectional")
@@
 			)
 			(layers "F.Cu" "F.Mask")
-			(net 58 "unconnected-(U1-GND-Pad38)")
+			(net 57 "unconnected-(U1-GND-Pad38)")
 			(pinfunction "GND")
 			(pintype "bidirectional")
@@
 			(layers "*.Cu" "*.Mask")
 			(remove_unused_layers no)
-			(net 64 "unconnected-(U1-GND-Pad42)")
+			(net 63 "unconnected-(U1-GND-Pad42)")
 			(pinfunction "GND")
 			(pintype "power_in")
@@
 			)
 			(layers "F.Cu" "F.Mask")
-			(net 64 "unconnected-(U1-GND-Pad42)")
+			(net 63 "unconnected-(U1-GND-Pad42)")
 			(pinfunction "GND")
 			(pintype "power_in")
@@
 		)
 	)
+	(footprint "MountingHole:MountingHole_3.2mm_M3"
+		(layer "F.Cu")
+		(at 3.475 3.475)
+		(descr "Mounting Hole 3.2mm, M3, no annular, generated by kicad-footprint-generator mountinghole.py")
+		(tags "mountinghole M3")
+		(property "Reference" "H4"
+			(at 0 -4.15 0)
+			(layer "F.SilkS")
+			(effects
+				(font
+					(size 1 1)
+					(thickness 0.15)
+				)
+			)
+		)
+		(property "Value" "MountingHole"
+			(at 0 4.15 0)
+			(layer "F.Fab")
+			(effects
+				(font
+					(size 1 1)
+					(thickness 0.15)
+				)
+			)
+		)
+		(property "Datasheet" "~"
+			(at 0 0 0)
+			(layer "F.Fab")
+			(hide yes)
+			(effects
+				(font
+					(size 1.27 1.27)
+					(thickness 0.15)
+				)
+			)
+		)
+		(property "Description" "Mounting Hole without connection"
+			(at 0 0 0)
+			(layer "F.Fab")
+			(hide yes)
+			(effects
+				(font
+					(size 1.27 1.27)
+					(thickness 0.15)
+				)
+			)
+		)
+		(property ki_fp_filters "MountingHole*")
+		(sheetname "/")
+		(sheetfile "pad.kicad_sch")
+		(attr exclude_from_pos_files exclude_from_bom)
+		(fp_circle
+			(center 0 0)
+			(end 3.2 0)
+			(stroke
+				(width 0.15)
+				(type solid)
+			)
+			(fill no)
+			(layer "Cmts.User")
+		)
+		(fp_circle
+			(center 0 0)
+			(end 3.45 0)
+			(stroke
+				(width 0.05)
+				(type solid)
+			)
+			(fill no)
+			(layer "F.CrtYd")
+		)
+		(fp_text user "${REFERENCE}"
+			(at 0 0 0)
+			(layer "F.Fab")
+			(effects
+				(font
+					(size 1 1)
+					(thickness 0.15)
+				)
+			)
+		)
+		(pad "" np_thru_hole circle
+			(at 0 0)
+			(size 3.2 3.2)
+			(drill 3.2)
+			(layers "*.Cu" "*.Mask")
+		)
+		(embedded_fonts no)
+	)
 	(footprint "ScottoKeebs_MX:MX_PCB_1.00u"
 		(layer "F.Cu")
@@
 	)
 	(segment
+		(start 246.371 122.011)
+		(end 246.371 187.779)
+		(width 0.2)
+		(layer "B.Cu")
+		(net 15)
+	)
+	(segment
 		(start 175.425 192.05)
 		(end 194.475 192.05)
@@
 	(segment
 		(start 246.371 187.779)
-		(end 246.371 119.471)
+		(end 232.575 201.575)
 		(width 0.2)
 		(layer "B.Cu")
@@
 	)
 	(segment
-		(start 246.371 119.471)
-		(end 245.22 118.32)
+		(start 245.22 120.86)
+		(end 246.371 122.011)
 		(width 0.2)
 		(layer "B.Cu")
@@
 		(width 0.2)
 		(layer "B.Cu")
-		(net 15)
-	)
-	(segment
-		(start 232.575 201.575)
-		(end 246.371 187.779)
-		(width 0.2)
-		(layer "B.Cu")
