File: pad/pad.kicad_sch (KiCad schematic)
At the start: 45 parts, among them J1 OLED_128x64, SW1 ESC, SW10 5, SW11 6, SW12 1, SW13 2, SW14 3, SW15 entrt, SW16 0, SW17 ., SW18 RotaryEncoder_Switch, SW19 RotaryEncoder_Switch, SW2 /, SW3 *, SW4 -, SW5 7, SW6 8, SW7 9, SW8 +, SW9 4, U1 Raspberry_Pi_Pico

Commit message: BOM
Connections:
- net Row5: now also U1.14 (GPIO10); no longer U1.13 (GND)
Changed lines of the file:
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@@
 	(global_label "Row5"
 		(shape input)
-		(at 191.77 69.85 180)
+		(at 191.77 72.39 180)
 		(fields_autoplaced yes)
 		(effects
@@
 		)
 		(property "Intersheetrefs" "${INTERSHEET_REFS}"
-			(at 183.8258 69.85 0)
+			(at 183.8258 72.39 0)
 			(effects
 				(font
