File: splitly/splitly.kicad_sch (KiCad schematic)
At the start: 46 parts, among them J1 OLED_128x32, SW1 SW_Push_45deg, SW10 SW_Push_45deg, SW11 SW_Push_45deg, SW12 SW_Push_45deg, SW13 SW_Push_45deg, SW14 SW_Push_45deg, SW15 SW_Push_45deg, SW16 SW_Push_45deg, SW17 SW_Push_45deg, SW18 SW_Push_45deg, SW19 SW_Push_45deg, SW2 SW_Push_45deg, SW20 SW_Push_45deg, SW21 SW_Push_45deg, SW3 SW_Push_45deg, SW4 SW_Push_45deg, SW5 SW_Push_45deg, SW6 SW_Push_45deg, SW7 SW_Push_45deg, SW8 SW_Push_45deg, SW9 SW_Push_45deg, U1 Nice_Nano_V2

Commit message: images
Other:
- note added: "Left_Keboard Matrix"
- note removed: "Right_Keboard Matrix"
Changed lines of the file:
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@@
 		)
 	)
-	(text "Right_Keboard Matrix"
+	(text "Left_Keboard Matrix"
 		(exclude_from_sim no)
 		(at 44.704 20.32 0)
